File: Ki_Cad/ESP_32_MacroPad.kicad_sch (KiCad schematic)
At the start: 0 parts

Commit message: slow progress unfortunately
Other:
- added sheet Connectors (Connectors.kicad_sch)
Changed lines of the file:
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@@
+	)
+	(sheet
+		(at 205.74 187.96)
+		(size 66.04 58.42)
+		(exclude_from_sim no)
+		(in_bom yes)
+		(on_board yes)
+		(dnp no)
+		(fields_autoplaced yes)
+		(stroke
+			(width 0.1524)
+			(type solid)
+		)
+		(fill
+			(color 0 0 0 0.0000)
+		)
+		(property "Sheetname" "Connectors"
+			(at 205.74 187.2484 0)
+			(effects
+				(font
+					(size 1.27 1.27)
+				)
+				(justify left bottom)
+			)
+		)
+		(property "Sheetfile" "Connectors.kicad_sch"
+			(at 205.74 246.9646 0)
+			(effects
+				(font
+					(size 1.27 1.27)
+				)
+				(justify left top)
+			)
+		)
+		(instances
+			(project "ESP_32_MacroPad"
+				(path "/fa2979d6-93e1-46a4-a1b3-a2c8f322786c"
+					(page "4")
+				)
+			)
+		)
 	)
 	(sheet
