File: Ki_Cad/esp32_micro.kicad_sch (KiCad schematic)
At the start: 1 part, among them U2 ESP32-C6-WROOM-1-N8

Commit message: slow progress unfortunately
Parts:
- added Q1, Q2: BC847BPDW1, Package_TO_SOT_SMD:SOT-363_SC-70-6, symbol Transistor_BJT:BC847BPDW1
- added R2, R3: 10k, PCM_Resistor_SMD_AKL:R_0603_1608Metric, symbol PCM_Resistor_US_AKL:R_0603
Connections:
- net GND: now reaches U2.1 (GND), U2.28 (GND), U2.29_1 (GND), U2.29_2 (GND), U2.29_3 (GND), U2.29_4 (GND), U2.29_5 (GND), U2.29_6 (GND), U2.29_7 (GND), U2.29_8 (GND), U2.29_9 (GND)
- net KB_LED_MATRIX: now reaches U2.10 (IO8)
- net IO9: now reaches U2.15 (IO9)
- net IO9: now also Q2.6 (C1)
- net +3.3V: now reaches U2.2 (3V3)
- net ESP_EN: now reaches U2.3 (EN)
- net ESP_EN: now also Q1.4 (E2)
- new net: Q2.2 (B1), R2.2
- new net: Q1.5 (B2), R3.2
- new net DTR: Q2.1 (E1), R3.1
- new net RTS: Q1.3 (C2), R2.1
Other:
- moved on the sheet: U2
